File: kudox-game/pcb/kicad_files/kudox_game.kicad_pcb (KiCad board)
At the start: 2 copper layers, 145.7 x 130.4 mm, 62 parts, among them K0 KEYSW, K1 KEYSW, K11 KEYSW, K12 KEYSW, K13 KEYSW, K14 KEYSW, K15 KEYSW, K2 KEYSW, K20 KEYSW, K21 KEYSW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

Commit message: [game] Modified outlines and silk backboard. (#1)
* Modified outlines and silk backboard.

* Remove obsoleted files.

* Modified logos and url of Kudox Game on silk.

* Modified kudox for gerbar files.
Parts:
- added G***: LOGO, myparts:qmk-badge, B.Cu at (171.6, 132.8)
- added G***: LOGO, kudox_game_footprints:kudox_game_logo, B.Cu at (152.7, 140.1)
- added REF***: OSHW-Logo2_14.6x12mm_SilkScreen, Symbols:OSHW-Symbol_8.9x8mm_SilkScreen, B.Cu at (90.8, 76.7)
- moved REF*** 26.5 mm to (90.8, 76.7)
Other:
- board text added: "https://github.com/kumaokobo/kudox-keyboard"
- board text removed: "https://github.com/kumaokobo/kudox-keyboard.git"
