File: kudox-game/pcb/kicad_files/kudox_game.kicad_pcb (KiCad board)
At the start: 2 copper layers, 145.7 x 130.4 mm, 62 parts, among them K0 KEYSW, K1 KEYSW, K11 KEYSW, K12 KEYSW, K13 KEYSW, K14 KEYSW, K15 KEYSW, K2 KEYSW, K20 KEYSW, K21 KEYSW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

Commit message: Modified outlines and silk backboard.
Parts:
- added G***: LOGO, myparts:qmk-badge, B.Cu at (171.6, 132.8)
- added G***: LOGO, kudox_game_footprints:kudox_game_logo, B.Cu at (152.7, 140.1)
- moved REF*** 26.5 mm to (90.8, 76.7)

Commit message: Modified logos and url of Kudox Game on silk.
Parts:
- added REF***: OSHW-Logo2_14.6x12mm_SilkScreen, Symbols:OSHW-Symbol_8.9x8mm_SilkScreen, B.Cu at (90.8, 76.7)
Other:
- board text added: "https://github.com/kumaokobo/kudox-keyboard"
- board text removed: "https://github.com/kumaokobo/kudox-keyboard.git"

Commit message: Modified the silks of Kudox Game PCB.
Parts:
- moved G*** 32.2 mm to (140.5, 124.6)
- moved G*** 11.1 mm to (140.7, 124.6)
- moved G*** 7.85 mm to (155.8, 132.9)
- moved G*** 7.47 mm to (153.9, 133.0)
- moved REF*** 1.65 mm to (90.8, 78.3), turned to 180 degrees
- moved REF*** 1.63 mm to (90.8, 78.3)
Other:
- board text added: "rev 1.0"
Changed lines of the file:
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@@
   (general
     (thickness 1.6)
-    (drawings 225)
+    (drawings 227)
     (tracks 459)
     (zones 0)
@@
   )
   (module Symbols:OSHW-Symbol_8.9x8mm_SilkScreen (layer B.Cu)
-    (at 90.82 76.7)
+    (at 90.8 78.35 180)
     (descr "Open Source Hardware Symbol")
     (tags "Logo Symbol OSHW")
     (attr virtual)
-    (fp_text reference REF*** (at 0 0) (layer F.SilkS) hide
+    (fp_text reference REF*** (at 0 0 180) (layer F.SilkS) hide
       (effects (font (size 1 1) (thickness 0.15)))
     )
-    (fp_text value OSHW-Logo2_14.6x12mm_SilkScreen (at 0.75 0) (layer B.Fab) hide
+    (fp_text value OSHW-Logo2_14.6x12mm_SilkScreen (at 0.75 0 180) (layer B.Fab) hide
       (effects (font (size 1 1) (thickness 0.15)) (justify mirror))
     )
@@
   )
   (module myparts:qmk-badge (layer B.Cu)
-    (at 171.64 132.76 180)
+    (at 140.5 124.6 180)
     (fp_text reference G*** (at 0 0) (layer F.SilkS) hide
       (effects (font (size 1.524 1.524) (thickness 0.3)))
@@
   )
   (module kudox_game_footprints:kudox_game_logo (layer B.Cu)
-    (at 152.71 140.12 180)
+    (at 155.8 132.9 180)
     (fp_text reference G*** (at 0 0) (layer F.SilkS) hide
       (effects (font (size 1.524 1.524) (thickness 0.3)))
@@
   )
   (module kudox_game_footprints:kudox_game_logo (layer F.Cu)
-    (at 152.3 140.3)
+    (at 153.9 133)
     (fp_text reference G*** (at 0 0) (layer F.SilkS) hide
       (effects (font (size 1.524 1.524) (thickness 0.3)))
@@
     (descr "tactile push button, 6x6mm e.g. PHAP33xx series, height=4.3mm")
     (tags "tact sw push 6mm")
-    (fp_text reference RST_SW1 (at 3.25 -2) (layer F.SilkS)
+    (fp_text reference RST_SW1 (at 8.6 2.3 90) (layer F.SilkS)
       (effects (font (size 1 1) (thickness 0.15)))
     )
@@
   )
   (module Symbols:OSHW-Symbol_8.9x8mm_SilkScreen (layer F.Cu)
-    (at 90.8 76.72)
+    (at 90.8 78.35)
     (descr "Open Source Hardware Symbol")
     (tags "Logo Symbol OSHW")
@@
   )
   (module myparts:qmk-badge (layer F.Cu)
-    (at 133.1 132.7)
+    (at 140.7 124.6)
     (fp_text reference G*** (at 0 0) (layer F.SilkS) hide
       (effects (font (size 1.524 1.524) (thickness 0.3)))
@@
       (xy -9.943822 -1.795852)) (layer F.SilkS) (width 0.01))
   )
-  (gr_text https://github.com/kumaokobo/kudox-keyboard (at 81.915 94.234 90) (layer B.SilkS)
+  (gr_text "rev 1.0" (at 124.2 130.7) (layer B.SilkS)
+    (effects (font (size 1.5 1.5) (thickness 0.15)) (justify mirror))
+  )
+  (gr_text "rev 1.0" (at 185.6 130.7) (layer F.SilkS)
+    (effects (font (size 1.5 1.5) (thickness 0.15)))
+  )
+  (gr_text https://github.com/kumaokobo/kudox-keyboard (at 157.7 139.5) (layer B.SilkS)
     (effects (font (size 1.5 1.5) (thickness 0.3)) (justify mirror))
   )
@@
   (gr_curve (pts (xy 215.953236 175.539138) (xy 215.953236 176.474922) (xy 215.194633 177.233524) (xy 214.25885 177.233524)) (layer Eco1.User) (width 0.1))
   (gr_line (start 111.7 67.3) (end 111.7 53.330035) (layer Eco1.User) (width 0.1))
-  (gr_text https://github.com/kumaokobo/kudox-keyboard (at 81.915 94.234 90) (layer F.SilkS)
+  (gr_text https://github.com/kumaokobo/kudox-keyboard (at 151.8 139.5) (layer F.SilkS)
     (effects (font (size 1.5 1.5) (thickness 0.3)))
   )
