File: kudox-game/pcb/kicad_files/kudox_game.sch (KiCad schematic (older format))
At the start: 60 parts, among them K0 KEYSW, K1 KEYSW, K10 KEYSW, K11 KEYSW, K12 KEYSW, K13 KEYSW, K14 KEYSW, K15 KEYSW, K2 KEYSW, K20 KEYSW, K21 KEYSW, K22 KEYSW, K23 KEYSW, K24 KEYSW, K25 KEYSW, K26 KEYSW, K3 KEYSW, K30 KEYSW, K31 KEYSW, K34 KEYSW, K35 KEYSW, K36 KEYSW, K4 KEYSW, K40 KEYSW, K45 KEYSW, K46 KEYSW, K5 KEYSW, U1 ProMicro

Commit message: [game] Modified outlines and silk backboard. (#1)
* Modified outlines and silk backboard.

* Remove obsoleted files.

* Modified logos and url of Kudox Game on silk.

* Modified kudox for gerbar files.
Parts:
- removed R1, R2: 4.7k, Keebio-Parts:Resistor-Compact, symbol R
- removed RGB_STRIP1: Conn_01x03, Pin_Headers:Pin_Header_Straight_1x03_Pitch2.54mm, symbol Conn_01x03
- removed TRRS1: Audio-Jack-4, Keebio-Parts:TRRS-PJ-320A-dual, symbol Audio-Jack-4
Connections:
- net SCL: no longer names the net of U1.6 (3/PD0)
- net SDA: no longer names the net of U1.5 (2/PD1)
- net rgb_data: no longer names the net of U1.1 (TX0/PD3)
- no-connect marks 4 -> 7
Other:
- moved on the sheet: RST_SW1
Changed lines of the file:
@@
 EESchema Schematic File Version 4
-LIBS:power
-LIBS:device
-LIBS:74xx
-LIBS:audio
-LIBS:interface
 LIBS:kudox_game-cache
 EELAYER 29 0
@@
 Sheet 1 1
 Title "Kudox Game keyboard"
-Date "2019-06-30"
+Date "2019-07-01"
 Rev "1.0"
 Comp ""
-Comment1 "designed by Inken"
-Comment2 "https://github.com/x1-"
+Comment1 "designed by x1 and inken"
+Comment2 "https://github.com/kumaokobo/kudox-keyboard"
 Comment3 ""
 Comment4 ""
@@
 $EndComp
 $Comp
-L Audio-Jack-4 TRRS1
-U 1 1 5A8087E2
-P 1100 3200
-F 0 "TRRS1" H 1050 3280 50  0000 C CNN
-F 1 "Audio-Jack-4" H 1220 2830 50  0000 C CNN
-F 2 "Keebio-Parts:TRRS-PJ-320A-dual" H 1350 3300 50  0001 C CNN
-F 3 "" H 1350 3300 50  0001 C CNN
-	1    1100 3200
-	1    0    0    -1
-$EndComp
-$Comp
-L Conn_01x03 RGB_STRIP1
-U 1 1 5A8088A7
-P 1750 4200
-F 0 "RGB_STRIP1" H 1750 4400 50  0000 C CNN
-F 1 "Conn_01x03" H 1750 4000 50  0000 C CNN
-F 2 "Pin_Headers:Pin_Header_Straight_1x03_Pitch2.54mm" H 1750 4200 50  0001 C CNN
-F 3 "" H 1750 4200 50  0001 C CNN
-	1    1750 4200
-	1    0    0    -1
-$EndComp
-$Comp
 L SW_PUSH RST_SW1
 U 1 1 5A808917
-P 1450 4750
-F 0 "RST_SW1" H 1600 4860 50  0000 C CNN
-F 1 "SW_PUSH" H 1450 4670 50  0000 C CNN
-F 2 "Buttons_Switches_ThroughHole:SW_PUSH_6mm_h4.3mm" H 1450 4750 60  0001 C CNN
-F 3 "" H 1450 4750 60  0000 C CNN
-	1    1450 4750
+P 2350 3400
+F 0 "RST_SW1" H 2500 3510 50  0000 C CNN
+F 1 "SW_PUSH" H 2350 3320 50  0000 C CNN
+F 2 "Buttons_Switches_ThroughHole:SW_PUSH_6mm_h4.3mm" H 2350 3400 60  0001 C CNN
+F 3 "" H 2350 3400 60  0000 C CNN
+	1    2350 3400
 	1    0    0    -1
 $EndComp
@@
 Wire Wire Line
 	3050 1800 3300 1800
-Text GLabel 1450 2100 0    60   Input ~ 0
-SCL
-Text GLabel 1450 2000 0    60   Input ~ 0
-SDA
-Wire Wire Line
-	1450 2000 1650 2000
-Wire Wire Line
-	1450 2100 1650 2100
 Text GLabel 3300 2100 2    60   Input ~ 0
 col0
@@
 	1450 2200 1650 2200
 NoConn ~ 3050 1600
-Text GLabel 1450 1600 0    60   Input ~ 0
-rgb_data
-Wire Wire Line
-	1450 1600 1650 1600
 NoConn ~ 1650 1700
 NoConn ~ 1650 2300
 NoConn ~ 3050 2000
-$Comp
-L GND #PWR03
-U 1 1 5A808DAF
-P 900 3600
-F 0 "#PWR03" H 900 3350 50  0001 C CNN
-F 1 "GND" H 900 3450 50  0000 C CNN
-F 2 "" H 900 3600 50  0001 C CNN
-F 3 "" H 900 3600 50  0001 C CNN
-	1    900  3600
-	1    0    0    -1
-$EndComp
-Text GLabel 1850 3200 2    60   Input ~ 0
-SDA
-Text GLabel 1850 3300 2    60   Input ~ 0
-SCL
-Wire Wire Line
-	1300 3200 1450 3200
-Wire Wire Line
-	1300 3300 1700 3300
-$Comp
-L GND #PWR04
-U 1 1 5A808EA3
-P 1550 4300
-F 0 "#PWR04" H 1550 4050 50  0001 C CNN
-F 1 "GND" H 1550 4150 50  0000 C CNN
-F 2 "" H 1550 4300 50  0001 C CNN
-F 3 "" H 1550 4300 50  0001 C CNN
-	1    1550 4300
-	0    1    1    0
-$EndComp
-$Comp
-L VCC #PWR05
-U 1 1 5A808EBA
-P 1550 4100
-F 0 "#PWR05" H 1550 3950 50  0001 C CNN
-F 1 "VCC" H 1550 4250 50  0000 C CNN
-F 2 "" H 1550 4100 50  0001 C CNN
-F 3 "" H 1550 4100 50  0001 C CNN
-	1    1550 4100
-	0    -1   -1   0
-$EndComp
-Text GLabel 1300 4200 0    60   Input ~ 0
-rgb_data
-Wire Wire Line
-	1300 4200 1550 4200
-Text GLabel 1150 4750 0    60   Input ~ 0
+Text GLabel 2050 3400 0    60   Input ~ 0
 RST
 $Comp
 L GND #PWR06
 U 1 1 5A80901B
-P 1750 4750
-F 0 "#PWR06" H 1750 4500 50  0001 C CNN
-F 1 "GND" H 1750 4600 50  0000 C CNN
-F 2 "" H 1750 4750 50  0001 C CNN
-F 3 "" H 1750 4750 50  0001 C CNN
-	1    1750 4750
+P 2650 3400
+F 0 "#PWR06" H 2650 3150 50  0001 C CNN
+F 1 "GND" H 2650 3250 50  0000 C CNN
+F 2 "" H 2650 3400 50  0001 C CNN
+F 3 "" H 2650 3400 50  0001 C CNN
+	1    2650 3400
 	0    -1   -1   0
 $EndComp
@@
 Text GLabel 10000 1350 1    60   Input ~ 0
 col6
-$Comp
-L R R1
-U 1 1 5A80A2DF
-P 1450 3350
-F 0 "R1" V 1530 3350 50  0000 C CNN
-F 1 "4.7k" V 1450 3350 50  0000 C CNN
-F 2 "Keebio-Parts:Resistor-Compact" V 1380 3350 50  0001 C CNN
-F 3 "" H 1450 3350 50  0001 C CNN
-	1    1450 3350
-	1    0    0    -1
-$EndComp
-$Comp
-L R R2
-U 1 1 5A80A522
-P 1700 3450
-F 0 "R2" V 1780 3450 50  0000 C CNN
-F 1 "4.7k" V 1700 3450 50  0000 C CNN
-F 2 "Keebio-Parts:Resistor-Compact" V 1630 3450 50  0001 C CNN
-F 3 "" H 1700 3450 50  0001 C CNN
-	1    1700 3450
-	1    0    0    -1
-$EndComp
-Connection ~ 1450 3200
-Connection ~ 1700 3300
-$Comp
-L VCC #PWR09
-U 1 1 5A80ACC6
-P 1900 3600
-F 0 "#PWR09" H 1900 3450 50  0001 C CNN
-F 1 "VCC" H 1900 3750 50  0000 C CNN
-F 2 "" H 1900 3600 50  0001 C CNN
-F 3 "" H 1900 3600 50  0001 C CNN
-	1    1900 3600
-	0    1    1    0
-$EndComp
-Wire Wire Line
-	1300 3400 1300 3600
-Wire Wire Line
-	1300 3600 1450 3600
-Wire Wire Line
-	1450 3500 1450 3600
-Connection ~ 1450 3600
-Connection ~ 1700 3600
 Wire Wire Line
 	5400 1900 6200 1900
@@
 Wire Wire Line
 	9200 2250 9200 2950
-Wire Wire Line
-	1450 3200 1850 3200
-Wire Wire Line
-	1700 3300 1850 3300
-Wire Wire Line
-	1450 3600 1700 3600
-Wire Wire Line
-	1700 3600 1900 3600
 Wire Wire Line
 	10000 1350 10000 2950
@@
 	0    -1   -1   0
 $EndComp
+NoConn ~ 1650 1600
+NoConn ~ 1650 2000
+NoConn ~ 1650 2100
 $EndSCHEMATC

Commit message: Modified the silks of Kudox Game PCB.
Parts:
- removed D10: D, Keebio-Parts:Diode-dual, symbol D
- removed K10: KEYSW, Keebio-Parts:Hybrid_PCB_100H_Dual_hole-nosilk, symbol KEYSW
Changed lines of the file:
@@
 Connection ~ 7800 1900
-$Comp
-L KEYSW K10
-U 1 1 5A809C1D
-P 4900 2250
-F 0 "K10" H 4850 2250 60  0000 C CNN
-F 1 "KEYSW" H 4900 2150 60  0001 C CNN
-F 2 "Keebio-Parts:Hybrid_PCB_100H_Dual_hole-nosilk" H 4900 2250 60  0001 C CNN
-F 3 "" H 4900 2250 60  0000 C CNN
-	1    4900 2250
-	1    0    0    -1
-$EndComp
-$Comp
-L D D10
-U 1 1 5A809C23
-P 4600 2500
-F 0 "D10" H 4600 2600 50  0000 C CNN
-F 1 "D" H 4600 2400 50  0000 C CNN
-F 2 "Keebio-Parts:Diode-dual" H 4600 2500 50  0001 C CNN
-F 3 "" H 4600 2500 50  0001 C CNN
-	1    4600 2500
-	0    -1   -1   0
-$EndComp
-Wire Wire Line
-	4600 2250 4600 2350
 $Comp
 L KEYSW K11
@@
 Wire Wire Line
 	8600 2250 8600 2350
-Wire Wire Line
-	4500 2650 4600 2650
 Connection ~ 5400 2650
 Connection ~ 6200 2650
@@
 	5200 1300 5200 1500
 Connection ~ 5200 1500
-Connection ~ 5200 2250
 Connection ~ 5200 2950
 Connection ~ 5200 3700
@@
 Connection ~ 6000 2950
 Connection ~ 4600 1900
-Connection ~ 4600 2650
 Connection ~ 4600 3350
 Connection ~ 4600 4100
@@
 	8600 3350 9400 3350
 Wire Wire Line
-	5200 1500 5200 2250
-Wire Wire Line
-	5200 2250 5200 2950
-Wire Wire Line
 	5200 2950 5200 3700
 Wire Wire Line
@@
 Wire Wire Line
 	4600 1900 5400 1900
-Wire Wire Line
-	4600 2650 5400 2650
 Wire Wire Line
 	4600 3350 5400 3350
@@
 NoConn ~ 1650 2000
 NoConn ~ 1650 2100
+Wire Wire Line
+	4500 2650 5400 2650
+Wire Wire Line
+	5200 1500 5200 2950
 $EndSCHEMATC

Commit message: Modified settings of KiCad libraries.
Parts:
- D0, D1, D11, D12, D13, D14, D15, D2, D20, D21, D22, D23, D24, D25, D26, D3, D30, D31, D34, D35, D36, D4, D40, D45, D46, D5: symbol D -> kudox-game-parts:D
- K0, K1, K11, K12, K13, K14, K15, K2, K20, K21, K22, K23, K24, K25, K26, K3, K30, K31, K34, K35, K36, K4, K40, K45, K46, K5: symbol KEYSW -> kudox-game-parts:KEYSW
- RST_SW1: symbol SW_PUSH -> kudox-game-parts:SW_PUSH
- U1: symbol ProMicro -> kudox-game-parts:ProMicro
Changed lines of the file:
@@
 $EndDescr
 $Comp
-L ProMicro U1
+L kudox-game-parts:ProMicro U1
 U 1 1 5A8086FE
 P 2350 2150
@@
 $EndComp
 $Comp
-L SW_PUSH RST_SW1
+L kudox-game-parts:SW_PUSH RST_SW1
 U 1 1 5A808917
 P 2350 3400
@@
 $EndComp
 $Comp
-L GND #PWR01
+L kudox-game-parts:GND #PWR01
 U 1 1 5A80895C
 P 3050 1700
@@
 $EndComp
 $Comp
-L VCC #PWR02
+L kudox-game-parts:VCC #PWR02
 U 1 1 5A808978
 P 3050 1900
@@
 RST
 $Comp
-L GND #PWR06
+L kudox-game-parts:GND #PWR06
 U 1 1 5A80901B
 P 2650 3400
@@
 $EndComp
 $Comp
-L GND #PWR07
+L kudox-game-parts:GND #PWR07
 U 1 1 5A8090D7
 P 1650 1800
@@
 $EndComp
 $Comp
-L GND #PWR08
+L kudox-game-parts:GND #PWR08
 U 1 1 5A8090EE
 P 1650 1900
@@
 $EndComp
 $Comp
-L KEYSW K0
+L kudox-game-parts:KEYSW K0
 U 1 1 5A808C37
 P 4900 1500
@@
 $EndComp
 $Comp
-L D D0
+L kudox-game-parts:D D0
 U 1 1 5A808D18
 P 4600 1750
@@
 	4600 1500 4600 1600
 $Comp
-L KEYSW K1
+L kudox-game-parts:KEYSW K1
 U 1 1 5A809089
 P 5700 1500
@@
 $EndComp
 $Comp
-L D D1
+L kudox-game-parts:D D1
 U 1 1 5A80908F
 P 5400 1750
@@
 	5400 1500 5400 1600
 $Comp
-L KEYSW K2
+L kudox-game-parts:KEYSW K2
 U 1 1 5A8091F6
 P 6500 1500
@@
 $EndComp
 $Comp
-L D D2
+L kudox-game-parts:D D2
 U 1 1 5A8091FC
 P 6200 1750
@@
 	6200 1500 6200 1600
 $Comp
-L KEYSW K3
+L kudox-game-parts:KEYSW K3
 U 1 1 5A809203
 P 7300 1500
@@
 $EndComp
 $Comp
-L D D3
+L kudox-game-parts:D D3
 U 1 1 5A809209
 P 7000 1750
@@
 	7000 1500 7000 1600
 $Comp
-L KEYSW K4
+L kudox-game-parts:KEYSW K4
 U 1 1 5A80948D
 P 8100 1500
@@
 $EndComp
 $Comp
-L D D4
+L kudox-game-parts:D D4
 U 1 1 5A809493
 P 7800 1750
@@
 	7800 1500 7800 1600
 $Comp
-L KEYSW K5
+L kudox-game-parts:KEYSW K5
 U 1 1 5A80949A
 P 8900 1500
@@
 $EndComp
 $Comp
-L D D5
+L kudox-game-parts:D D5
 U 1 1 5A8094A0
 P 8600 1750
@@
 Connection ~ 7800 1900
 $Comp
-L KEYSW K11
+L kudox-game-parts:KEYSW K11
 U 1 1 5A809C2A
 P 5700 2250
@@
 $EndComp
 $Comp
-L D D11
+L kudox-game-parts:D D11
 U 1 1 5A809C30
 P 5400 2500
@@
 	5400 2250 5400 2350
 $Comp
-L KEYSW K12
+L kudox-game-parts:KEYSW K12
 U 1 1 5A809C37
 P 6500 2250
@@
 $EndComp
 $Comp
-L D D12
+L kudox-game-parts:D D12
 U 1 1 5A809C3D
 P 6200 2500
@@
 	6200 2250 6200 2350
 $Comp
-L KEYSW K13
+L kudox-game-parts:KEYSW K13
 U 1 1 5A809C44
 P 7300 2250
@@
 $EndComp
 $Comp
-L D D13
+L kudox-game-parts:D D13
 U 1 1 5A809C4A
 P 7000 2500
@@
 	7000 2250 7000 2350
 $Comp
-L KEYSW K14
+L kudox-game-parts:KEYSW K14
 U 1 1 5A809C51
 P 8100 2250
@@
 $EndComp
 $Comp
-L D D14
+L kudox-game-parts:D D14
 U 1 1 5A809C57
 P 7800 2500
@@
 	7800 2250 7800 2350
 $Comp
-L KEYSW K15
+L kudox-game-parts:KEYSW K15
 U 1 1 5A809C5E
 P 8900 2250
@@
 $EndComp
 $Comp
-L D D15
+L kudox-game-parts:D D15
 U 1 1 5A809C64
 P 8600 2500
@@
 Connection ~ 7800 2650
 $Comp
-L KEYSW K20
+L kudox-game-parts:KEYSW K20
 U 1 1 5A80AB8A
 P 4900 2950
@@
 $EndComp
 $Comp
-L D D20
+L kudox-game-parts:D D20
 U 1 1 5A80AB90
 P 4600 3200
@@
 	4600 2950 4600 3050
 $Comp
-L KEYSW K21
+L kudox-game-parts:KEYSW K21
 U 1 1 5A80AB97
 P 5700 2950
@@
 $EndComp
 $Comp
-L D D21
+L kudox-game-parts:D D21
 U 1 1 5A80AB9D
 P 5400 3200
@@
 	5400 2950 5400 3050
 $Comp
-L KEYSW K22
+L kudox-game-parts:KEYSW K22
 U 1 1 5A80ABA4
 P 6500 2950
@@
 $EndComp
 $Comp
-L D D22
+L kudox-game-parts:D D22
 U 1 1 5A80ABAA
 P 6200 3200
@@
 	6200 2950 6200 3050
 $Comp
-L KEYSW K23
+L kudox-game-parts:KEYSW K23
 U 1 1 5A80ABB1
 P 7300 2950
@@
 $EndComp
 $Comp
-L D D23
+L kudox-game-parts:D D23
 U 1 1 5A80ABB7
 P 7000 3200
@@
 	7000 2950 7000 3050
 $Comp
-L KEYSW K24
+L kudox-game-parts:KEYSW K24
 U 1 1 5A80ABBE
 P 8100 2950
@@
 $EndComp
 $Comp
-L D D24
+L kudox-game-parts:D D24
 U 1 1 5A80ABC4
 P 7800 3200
@@
 	7800 2950 7800 3050
 $Comp
-L KEYSW K25
+L kudox-game-parts:KEYSW K25
 U 1 1 5A80ABCB
 P 8900 2950
@@
 $EndComp
 $Comp
-L D D25
+L kudox-game-parts:D D25
 U 1 1 5A80ABD1
 P 8600 3200
@@
 	8600 2950 8600 3050
 $Comp
-L KEYSW K26
+L kudox-game-parts:KEYSW K26
 U 1 1 5A80ABD8
 P 9700 2950
@@
 $EndComp
 $Comp
-L D D26
+L kudox-game-parts:D D26
 U 1 1 5A80ABDE
 P 9400 3200
@@
 Connection ~ 8600 3350
 $Comp
-L KEYSW K30
+L kudox-game-parts:KEYSW K30
 U 1 1 5A80ABEB
 P 4900 3700
@@
 $EndComp
 $Comp
-L D D30
+L kudox-game-parts:D D30
 U 1 1 5A80ABF1
 P 4600 3950
@@
 	4600 3700 4600 3800
 $Comp
-L KEYSW K31
+L kudox-game-parts:KEYSW K31
 U 1 1 5A80ABF8
 P 5700 3700
@@
 $EndComp
 $Comp
-L D D31
+L kudox-game-parts:D D31
 U 1 1 5A80ABFE
 P 5400 3950
@@
 	5400 3700 5400 3800
 $Comp
-L KEYSW K34
+L kudox-game-parts:KEYSW K34
 U 1 1 5A80AC1F
 P 8100 3700
@@
 $EndComp
 $Comp
-L D D34
+L kudox-game-parts:D D34
 U 1 1 5A80AC25
 P 7800 3950
@@
 Connection ~ 5400 4100
 $Comp
-L KEYSW K40
+L kudox-game-parts:KEYSW K40
 U 1 1 5A80E493
 P 4900 4500
@@
 $EndComp
 $Comp
-L D D40
+L kudox-game-parts:D D40
 U 1 1 5A80E499
 P 4600 4750
@@
 	4600 4500 4600 4600
 $Comp
-L KEYSW K46
+L kudox-game-parts:KEYSW K46
 U 1 1 5A80E4E1
 P 9700 4500
@@
 $EndComp
 $Comp
-L D D46
+L kudox-game-parts:D D46
 U 1 1 5A80E4E7
 P 9400 4750
@@
 Connection ~ 9200 3700
 $Comp
-L KEYSW K35
+L kudox-game-parts:KEYSW K35
 U 1 1 5A80AC2C
 P 8900 3700
@@
 $EndComp
 $Comp
-L D D35
+L kudox-game-parts:D D35
 U 1 1 5A80AC32
 P 8600 3950
@@
 Connection ~ 10000 3700
 $Comp
-L KEYSW K36
+L kudox-game-parts:KEYSW K36
 U 1 1 5A80AC39
 P 9700 3700
@@
 $EndComp
 $Comp
-L D D36
+L kudox-game-parts:D D36
 U 1 1 5A80AC3F
 P 9400 3950
@@
 	8600 4500 8600 4600
 $Comp
-L KEYSW K45
+L kudox-game-parts:KEYSW K45
 U 1 1 5A80E4D4
 P 8900 4500
@@
 Connection ~ 8600 4900
 $Comp
-L D D45
+L kudox-game-parts:D D45
 U 1 1 5A80E4DA
 P 8600 4750
