File: kudox-game/rev2/kudox_game.sch (KiCad schematic (older format))
At the start: 55 parts, among them K0 KEYSW, K1 KEYSW, K11 KEYSW, K12 KEYSW, K13 KEYSW, K14 KEYSW, K15 KEYSW, K2 KEYSW, K20 KEYSW, K21 KEYSW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

Commit message: [kudox-game] Modify Kudox Game rev2 using MX socket optional switch foot print. (#45)
Parts:
- K0, K1, K11, K12, K13, K14, K15, K2, K20, K21, K22, K23, K24, K25, K26, K3, K31, K34, K35, K36, K4, K5: footprint kudox_game_footprints:Mx_hotswappable -> kudox_game_footprints:MX_socket_optional_100
- K30, K40, K45: footprint kudox_game_footprints:Mx_hotswappable -> kudox_game_footprints:MX_socket_optional_150
- K46: footprint kudox_game_footprints:Mx_hotswappable -> kudox_game_footprints:MX_socket_optional_200
Changed lines of the file:
@@
 F 0 "K0" H 4850 1500 60  0000 C CNN
 F 1 "KEYSW" H 4900 1400 60  0001 C CNN
-F 2 "kudox_game_footprints:Mx_hotswappable" H 4900 1500 60  0001 C CNN
+F 2 "kudox_game_footprints:MX_socket_optional_100" H 4900 1500 60  0001 C CNN
 F 3 "" H 4900 1500 60  0000 C CNN
 	1    4900 1500
@@
 F 0 "K1" H 5650 1500 60  0000 C CNN
 F 1 "KEYSW" H 5700 1400 60  0001 C CNN
-F 2 "kudox_game_footprints:Mx_hotswappable" H 5700 1500 60  0001 C CNN
+F 2 "kudox_game_footprints:MX_socket_optional_100" H 5700 1500 60  0001 C CNN
 F 3 "" H 5700 1500 60  0000 C CNN
 	1    5700 1500
@@
 F 0 "K2" H 6450 1500 60  0000 C CNN
 F 1 "KEYSW" H 6500 1400 60  0001 C CNN
-F 2 "kudox_game_footprints:Mx_hotswappable" H 6500 1500 60  0001 C CNN
+F 2 "kudox_game_footprints:MX_socket_optional_100" H 6500 1500 60  0001 C CNN
 F 3 "" H 6500 1500 60  0000 C CNN
 	1    6500 1500
@@
 F 0 "K3" H 7250 1500 60  0000 C CNN
 F 1 "KEYSW" H 7300 1400 60  0001 C CNN
-F 2 "kudox_game_footprints:Mx_hotswappable" H 7300 1500 60  0001 C CNN
+F 2 "kudox_game_footprints:MX_socket_optional_100" H 7300 1500 60  0001 C CNN
 F 3 "" H 7300 1500 60  0000 C CNN
 	1    7300 1500
@@
 F 0 "K4" H 8050 1500 60  0000 C CNN
 F 1 "KEYSW" H 8100 1400 60  0001 C CNN
-F 2 "kudox_game_footprints:Mx_hotswappable" H 8100 1500 60  0001 C CNN
+F 2 "kudox_game_footprints:MX_socket_optional_100" H 8100 1500 60  0001 C CNN
 F 3 "" H 8100 1500 60  0000 C CNN
 	1    8100 1500
@@
 F 0 "K5" H 8850 1500 60  0000 C CNN
 F 1 "KEYSW" H 8900 1400 60  0001 C CNN
-F 2 "kudox_game_footprints:Mx_hotswappable" H 8900 1500 60  0001 C CNN
+F 2 "kudox_game_footprints:MX_socket_optional_100" H 8900 1500 60  0001 C CNN
 F 3 "" H 8900 1500 60  0000 C CNN
 	1    8900 1500
@@
 F 0 "K11" H 5650 2250 60  0000 C CNN
 F 1 "KEYSW" H 5700 2150 60  0001 C CNN
-F 2 "kudox_game_footprints:Mx_hotswappable" H 5700 2250 60  0001 C CNN
+F 2 "kudox_game_footprints:MX_socket_optional_100" H 5700 2250 60  0001 C CNN
 F 3 "" H 5700 2250 60  0000 C CNN
 	1    5700 2250
@@
 F 0 "K12" H 6450 2250 60  0000 C CNN
 F 1 "KEYSW" H 6500 2150 60  0001 C CNN
-F 2 "kudox_game_footprints:Mx_hotswappable" H 6500 2250 60  0001 C CNN
+F 2 "kudox_game_footprints:MX_socket_optional_100" H 6500 2250 60  0001 C CNN
 F 3 "" H 6500 2250 60  0000 C CNN
 	1    6500 2250
@@
 F 0 "K13" H 7250 2250 60  0000 C CNN
 F 1 "KEYSW" H 7300 2150 60  0001 C CNN
-F 2 "kudox_game_footprints:Mx_hotswappable" H 7300 2250 60  0001 C CNN
+F 2 "kudox_game_footprints:MX_socket_optional_100" H 7300 2250 60  0001 C CNN
 F 3 "" H 7300 2250 60  0000 C CNN
 	1    7300 2250
@@
 F 0 "K14" H 8050 2250 60  0000 C CNN
 F 1 "KEYSW" H 8100 2150 60  0001 C CNN
-F 2 "kudox_game_footprints:Mx_hotswappable" H 8100 2250 60  0001 C CNN
+F 2 "kudox_game_footprints:MX_socket_optional_100" H 8100 2250 60  0001 C CNN
 F 3 "" H 8100 2250 60  0000 C CNN
 	1    8100 2250
@@
 F 0 "K15" H 8850 2250 60  0000 C CNN
 F 1 "KEYSW" H 8900 2150 60  0001 C CNN
-F 2 "kudox_game_footprints:Mx_hotswappable" H 8900 2250 60  0001 C CNN
+F 2 "kudox_game_footprints:MX_socket_optional_100" H 8900 2250 60  0001 C CNN
 F 3 "" H 8900 2250 60  0000 C CNN
 	1    8900 2250
@@
 F 0 "K20" H 4850 2950 60  0000 C CNN
 F 1 "KEYSW" H 4900 2850 60  0001 C CNN
-F 2 "kudox_game_footprints:Mx_hotswappable" H 4900 2950 60  0001 C CNN
+F 2 "kudox_game_footprints:MX_socket_optional_100" H 4900 2950 60  0001 C CNN
 F 3 "" H 4900 2950 60  0000 C CNN
 	1    4900 2950
@@
 F 0 "K21" H 5650 2950 60  0000 C CNN
 F 1 "KEYSW" H 5700 2850 60  0001 C CNN
-F 2 "kudox_game_footprints:Mx_hotswappable" H 5700 2950 60  0001 C CNN
+F 2 "kudox_game_footprints:MX_socket_optional_100" H 5700 2950 60  0001 C CNN
 F 3 "" H 5700 2950 60  0000 C CNN
 	1    5700 2950
@@
 F 0 "K22" H 6450 2950 60  0000 C CNN
 F 1 "KEYSW" H 6500 2850 60  0001 C CNN
-F 2 "kudox_game_footprints:Mx_hotswappable" H 6500 2950 60  0001 C CNN
+F 2 "kudox_game_footprints:MX_socket_optional_100" H 6500 2950 60  0001 C CNN
 F 3 "" H 6500 2950 60  0000 C CNN
 	1    6500 2950
@@
 F 0 "K23" H 7250 2950 60  0000 C CNN
 F 1 "KEYSW" H 7300 2850 60  0001 C CNN
-F 2 "kudox_game_footprints:Mx_hotswappable" H 7300 2950 60  0001 C CNN
+F 2 "kudox_game_footprints:MX_socket_optional_100" H 7300 2950 60  0001 C CNN
 F 3 "" H 7300 2950 60  0000 C CNN
 	1    7300 2950
@@
 F 0 "K24" H 8050 2950 60  0000 C CNN
 F 1 "KEYSW" H 8100 2850 60  0001 C CNN
-F 2 "kudox_game_footprints:Mx_hotswappable" H 8100 2950 60  0001 C CNN
+F 2 "kudox_game_footprints:MX_socket_optional_100" H 8100 2950 60  0001 C CNN
 F 3 "" H 8100 2950 60  0000 C CNN
 	1    8100 2950
@@
 F 0 "K25" H 8850 2950 60  0000 C CNN
 F 1 "KEYSW" H 8900 2850 60  0001 C CNN
-F 2 "kudox_game_footprints:Mx_hotswappable" H 8900 2950 60  0001 C CNN
+F 2 "kudox_game_footprints:MX_socket_optional_100" H 8900 2950 60  0001 C CNN
 F 3 "" H 8900 2950 60  0000 C CNN
 	1    8900 2950
@@
 F 0 "K26" H 9650 2950 60  0000 C CNN
 F 1 "KEYSW" H 9700 2850 60  0001 C CNN
-F 2 "kudox_game_footprints:Mx_hotswappable" H 9700 2950 60  0001 C CNN
+F 2 "kudox_game_footprints:MX_socket_optional_100" H 9700 2950 60  0001 C CNN
 F 3 "" H 9700 2950 60  0000 C CNN
 	1    9700 2950
@@
 F 0 "K30" H 4850 3700 60  0000 C CNN
 F 1 "KEYSW" H 4900 3600 60  0001 C CNN
-F 2 "kudox_game_footprints:Mx_hotswappable" H 4900 3700 60  0001 C CNN
+F 2 "kudox_game_footprints:MX_socket_optional_150" H 4900 3700 60  0001 C CNN
 F 3 "" H 4900 3700 60  0000 C CNN
 	1    4900 3700
@@
 F 0 "K31" H 5650 3700 60  0000 C CNN
 F 1 "KEYSW" H 5700 3600 60  0001 C CNN
-F 2 "kudox_game_footprints:Mx_hotswappable" H 5700 3700 60  0001 C CNN
+F 2 "kudox_game_footprints:MX_socket_optional_100" H 5700 3700 60  0001 C CNN
 F 3 "" H 5700 3700 60  0000 C CNN
 	1    5700 3700
@@
 F 0 "K34" H 8050 3700 60  0000 C CNN
 F 1 "KEYSW" H 8100 3600 60  0001 C CNN
-F 2 "kudox_game_footprints:Mx_hotswappable" H 8100 3700 60  0001 C CNN
+F 2 "kudox_game_footprints:MX_socket_optional_100" H 8100 3700 60  0001 C CNN
 F 3 "" H 8100 3700 60  0000 C CNN
 	1    8100 3700
@@
 F 0 "K40" H 4850 4500 60  0000 C CNN
 F 1 "KEYSW" H 4900 4400 60  0001 C CNN
-F 2 "kudox_game_footprints:Mx_hotswappable" H 4900 4500 60  0001 C CNN
+F 2 "kudox_game_footprints:MX_socket_optional_150" H 4900 4500 60  0001 C CNN
 F 3 "" H 4900 4500 60  0000 C CNN
 	1    4900 4500
@@
 F 0 "K46" H 9650 4500 60  0000 C CNN
 F 1 "KEYSW" H 9700 4400 60  0001 C CNN
-F 2 "kudox_game_footprints:Mx_hotswappable" H 9700 4500 60  0001 C CNN
+F 2 "kudox_game_footprints:MX_socket_optional_200" H 9700 4500 60  0001 C CNN
 F 3 "" H 9700 4500 60  0000 C CNN
 	1    9700 4500
@@
 F 0 "K35" H 8850 3700 60  0000 C CNN
 F 1 "KEYSW" H 8900 3600 60  0001 C CNN
-F 2 "kudox_game_footprints:Mx_hotswappable" H 8900 3700 60  0001 C CNN
+F 2 "kudox_game_footprints:MX_socket_optional_100" H 8900 3700 60  0001 C CNN
 F 3 "" H 8900 3700 60  0000 C CNN
 	1    8900 3700
@@
 F 0 "K36" H 9650 3700 60  0000 C CNN
 F 1 "KEYSW" H 9700 3600 60  0001 C CNN
-F 2 "kudox_game_footprints:Mx_hotswappable" H 9700 3700 60  0001 C CNN
+F 2 "kudox_game_footprints:MX_socket_optional_100" H 9700 3700 60  0001 C CNN
 F 3 "" H 9700 3700 60  0000 C CNN
 	1    9700 3700
@@
 F 0 "K45" H 8850 4500 60  0000 C CNN
 F 1 "KEYSW" H 8900 4400 60  0001 C CNN
-F 2 "kudox_game_footprints:Mx_hotswappable" H 8900 4500 60  0001 C CNN
+F 2 "kudox_game_footprints:MX_socket_optional_150" H 8900 4500 60  0001 C CNN
 F 3 "" H 8900 4500 60  0000 C CNN
 	1    8900 4500
