File: kudox-columner/rev1/kudox-columner.sch (KiCad schematic (older format))
At the start: 72 parts, among them K0 KEYSW, K1 KEYSW, K10 KEYSW, K11 KEYSW, K12 KEYSW, K13 KEYSW, K14 KEYSW, K15 KEYSW, K16 KEYSW, K2 KEYSW, K20 KEYSW, K21 KEYSW, K22 KEYSW, K23 KEYSW, K24 KEYSW, K25 KEYSW, K3 KEYSW, K30 KEYSW, K31 KEYSW, K32 KEYSW, K33 KEYSW, K34 KEYSW, K35 KEYSW, K4 KEYSW, K40 KEYSW, K41 KEYSW, K42 KEYSW, K43 KEYSW, K44 KEYSW, K45 KEYSW, K46 KEYSW, K5 KEYSW, K6 KEYSW, U1 ProMicro

Commit message: Modify kudox-columner to add RGB pad
Parts:
- added J1, J2: RGB, kudox_footprints:pad_1x1, symbol Connector_Generic:Conn_01x01
- K0, K1, K10, K11, K12, K13, K14, K15, K16, K2, K20, K21, K22, K23, K24, K25, K3, K30, K31, K32, K33, K34, K35, K4, K40, K41, K42, K43, K44, K45, K46: footprint kudox_footprints:Mx_hotswappable -> kudox_footprints:MX_reversible_100
- RGB_STRIP1: footprint kudox_footprints:Pin_Header_Straight_1x03_Pitch2.54mm -> kudox_footprints:RGB-Strip
Connections:
- net SDA: now also J1.1 (Pin_1), J2.1 (Pin_1)
Changed lines of the file:
@@
 EESchema Schematic File Version 4
-LIBS:kudox-columner-cache
-EELAYER 29 0
+EELAYER 30 0
 EELAYER END
 $Descr A4 11693 8268
@@
 Sheet 1 1
 Title "Kudox Columner keyboard"
-Date "2019-10-01"
-Rev "1.0"
+Date "2021-07-21"
+Rev "1.2"
 Comp ""
 Comment1 "designed by x1 and inken"
@@
 F 0 "RGB_STRIP1" H 1750 4400 50  0000 C CNN
 F 1 "Conn_01x03" H 1750 4000 50  0000 C CNN
-F 2 "kudox_footprints:Pin_Header_Straight_1x03_Pitch2.54mm" H 1750 4200 50  0001 C CNN
+F 2 "kudox_footprints:RGB-Strip" H 1750 4200 50  0001 C CNN
 F 3 "" H 1750 4200 50  0001 C CNN
 	1    1750 4200
@@
 F 0 "K0" H 4850 1500 60  0000 C CNN
 F 1 "KEYSW" H 4900 1400 60  0001 C CNN
-F 2 "kudox_footprints:Mx_hotswappable" H 4900 1500 60  0001 C CNN
+F 2 "kudox_footprints:MX_reversible_100" H 4900 1500 60  0001 C CNN
 F 3 "" H 4900 1500 60  0000 C CNN
 	1    4900 1500
@@
 F 0 "K1" H 5650 1500 60  0000 C CNN
 F 1 "KEYSW" H 5700 1400 60  0001 C CNN
-F 2 "kudox_footprints:Mx_hotswappable" H 5700 1500 60  0001 C CNN
+F 2 "kudox_footprints:MX_reversible_100" H 5700 1500 60  0001 C CNN
 F 3 "" H 5700 1500 60  0000 C CNN
 	1    5700 1500
@@
 F 0 "K2" H 6450 1500 60  0000 C CNN
 F 1 "KEYSW" H 6500 1400 60  0001 C CNN
-F 2 "kudox_footprints:Mx_hotswappable" H 6500 1500 60  0001 C CNN
+F 2 "kudox_footprints:MX_reversible_100" H 6500 1500 60  0001 C CNN
 F 3 "" H 6500 1500 60  0000 C CNN
 	1    6500 1500
@@
 F 0 "K3" H 7250 1500 60  0000 C CNN
 F 1 "KEYSW" H 7300 1400 60  0001 C CNN
-F 2 "kudox_footprints:Mx_hotswappable" H 7300 1500 60  0001 C CNN
+F 2 "kudox_footprints:MX_reversible_100" H 7300 1500 60  0001 C CNN
 F 3 "" H 7300 1500 60  0000 C CNN
 	1    7300 1500
@@
 F 0 "K4" H 8050 1500 60  0000 C CNN
 F 1 "KEYSW" H 8100 1400 60  0001 C CNN
-F 2 "kudox_footprints:Mx_hotswappable" H 8100 1500 60  0001 C CNN
+F 2 "kudox_footprints:MX_reversible_100" H 8100 1500 60  0001 C CNN
 F 3 "" H 8100 1500 60  0000 C CNN
 	1    8100 1500
@@
 F 0 "K10" H 4850 2250 60  0000 C CNN
 F 1 "KEYSW" H 4900 2150 60  0001 C CNN
-F 2 "kudox_footprints:Mx_hotswappable" H 4900 2250 60  0001 C CNN
+F 2 "kudox_footprints:MX_reversible_100" H 4900 2250 60  0001 C CNN
 F 3 "" H 4900 2250 60  0000 C CNN
 	1    4900 2250
@@
 F 0 "K11" H 5650 2250 60  0000 C CNN
 F 1 "KEYSW" H 5700 2150 60  0001 C CNN
-F 2 "kudox_footprints:Mx_hotswappable" H 5700 2250 60  0001 C CNN
+F 2 "kudox_footprints:MX_reversible_100" H 5700 2250 60  0001 C CNN
 F 3 "" H 5700 2250 60  0000 C CNN
 	1    5700 2250
@@
 F 0 "K12" H 6450 2250 60  0000 C CNN
 F 1 "KEYSW" H 6500 2150 60  0001 C CNN
-F 2 "kudox_footprints:Mx_hotswappable" H 6500 2250 60  0001 C CNN
+F 2 "kudox_footprints:MX_reversible_100" H 6500 2250 60  0001 C CNN
 F 3 "" H 6500 2250 60  0000 C CNN
 	1    6500 2250
@@
 F 0 "K13" H 7250 2250 60  0000 C CNN
 F 1 "KEYSW" H 7300 2150 60  0001 C CNN
-F 2 "kudox_footprints:Mx_hotswappable" H 7300 2250 60  0001 C CNN
+F 2 "kudox_footprints:MX_reversible_100" H 7300 2250 60  0001 C CNN
 F 3 "" H 7300 2250 60  0000 C CNN
 	1    7300 2250
@@
 F 0 "K14" H 8050 2250 60  0000 C CNN
 F 1 "KEYSW" H 8100 2150 60  0001 C CNN
-F 2 "kudox_footprints:Mx_hotswappable" H 8100 2250 60  0001 C CNN
+F 2 "kudox_footprints:MX_reversible_100" H 8100 2250 60  0001 C CNN
 F 3 "" H 8100 2250 60  0000 C CNN
 	1    8100 2250
@@
 F 0 "K15" H 8850 2250 60  0000 C CNN
 F 1 "KEYSW" H 8900 2150 60  0001 C CNN
-F 2 "kudox_footprints:Mx_hotswappable" H 8900 2250 60  0001 C CNN
+F 2 "kudox_footprints:MX_reversible_100" H 8900 2250 60  0001 C CNN
 F 3 "" H 8900 2250 60  0000 C CNN
 	1    8900 2250
@@
 F 0 "K16" H 9650 2250 60  0000 C CNN
 F 1 "KEYSW" H 9700 2150 60  0001 C CNN
-F 2 "kudox_footprints:Mx_hotswappable" H 9700 2250 60  0001 C CNN
+F 2 "kudox_footprints:MX_reversible_100" H 9700 2250 60  0001 C CNN
 F 3 "" H 9700 2250 60  0000 C CNN
 	1    9700 2250
@@
 F 0 "K20" H 4850 2950 60  0000 C CNN
 F 1 "KEYSW" H 4900 2850 60  0001 C CNN
-F 2 "kudox_footprints:Mx_hotswappable" H 4900 2950 60  0001 C CNN
+F 2 "kudox_footprints:MX_reversible_100" H 4900 2950 60  0001 C CNN
 F 3 "" H 4900 2950 60  0000 C CNN
 	1    4900 2950
@@
 F 0 "K21" H 5650 2950 60  0000 C CNN
 F 1 "KEYSW" H 5700 2850 60  0001 C CNN
-F 2 "kudox_footprints:Mx_hotswappable" H 5700 2950 60  0001 C CNN
+F 2 "kudox_footprints:MX_reversible_100" H 5700 2950 60  0001 C CNN
 F 3 "" H 5700 2950 60  0000 C CNN
 	1    5700 2950
@@
 F 0 "K22" H 6450 2950 60  0000 C CNN
 F 1 "KEYSW" H 6500 2850 60  0001 C CNN
-F 2 "kudox_footprints:Mx_hotswappable" H 6500 2950 60  0001 C CNN
+F 2 "kudox_footprints:MX_reversible_100" H 6500 2950 60  0001 C CNN
 F 3 "" H 6500 2950 60  0000 C CNN
 	1    6500 2950
@@
 F 0 "K23" H 7250 2950 60  0000 C CNN
 F 1 "KEYSW" H 7300 2850 60  0001 C CNN
-F 2 "kudox_footprints:Mx_hotswappable" H 7300 2950 60  0001 C CNN
+F 2 "kudox_footprints:MX_reversible_100" H 7300 2950 60  0001 C CNN
 F 3 "" H 7300 2950 60  0000 C CNN
 	1    7300 2950
@@
 F 0 "K24" H 8050 2950 60  0000 C CNN
 F 1 "KEYSW" H 8100 2850 60  0001 C CNN
-F 2 "kudox_footprints:Mx_hotswappable" H 8100 2950 60  0001 C CNN
+F 2 "kudox_footprints:MX_reversible_100" H 8100 2950 60  0001 C CNN
 F 3 "" H 8100 2950 60  0000 C CNN
 	1    8100 2950
@@
 F 0 "K25" H 8850 2950 60  0000 C CNN
 F 1 "KEYSW" H 8900 2850 60  0001 C CNN
-F 2 "kudox_footprints:Mx_hotswappable" H 8900 2950 60  0001 C CNN
+F 2 "kudox_footprints:MX_reversible_100" H 8900 2950 60  0001 C CNN
 F 3 "" H 8900 2950 60  0000 C CNN
 	1    8900 2950
@@
 F 0 "K30" H 4850 3700 60  0000 C CNN
 F 1 "KEYSW" H 4900 3600 60  0001 C CNN
-F 2 "kudox_footprints:Mx_hotswappable" H 4900 3700 60  0001 C CNN
+F 2 "kudox_footprints:MX_reversible_100" H 4900 3700 60  0001 C CNN
 F 3 "" H 4900 3700 60  0000 C CNN
 	1    4900 3700
@@
 F 0 "K31" H 5650 3700 60  0000 C CNN
 F 1 "KEYSW" H 5700 3600 60  0001 C CNN
-F 2 "kudox_footprints:Mx_hotswappable" H 5700 3700 60  0001 C CNN
+F 2 "kudox_footprints:MX_reversible_100" H 5700 3700 60  0001 C CNN
 F 3 "" H 5700 3700 60  0000 C CNN
 	1    5700 3700
@@
 F 0 "K32" H 6450 3700 60  0000 C CNN
 F 1 "KEYSW" H 6500 3600 60  0001 C CNN
-F 2 "kudox_footprints:Mx_hotswappable" H 6500 3700 60  0001 C CNN
+F 2 "kudox_footprints:MX_reversible_100" H 6500 3700 60  0001 C CNN
 F 3 "" H 6500 3700 60  0000 C CNN
 	1    6500 3700
@@
 F 0 "K33" H 7250 3700 60  0000 C CNN
 F 1 "KEYSW" H 7300 3600 60  0001 C CNN
-F 2 "kudox_footprints:Mx_hotswappable" H 7300 3700 60  0001 C CNN
+F 2 "kudox_footprints:MX_reversible_100" H 7300 3700 60  0001 C CNN
 F 3 "" H 7300 3700 60  0000 C CNN
 	1    7300 3700
@@
 F 0 "K34" H 8050 3700 60  0000 C CNN
 F 1 "KEYSW" H 8100 3600 60  0001 C CNN
-F 2 "kudox_footprints:Mx_hotswappable" H 8100 3700 60  0001 C CNN
+F 2 "kudox_footprints:MX_reversible_100" H 8100 3700 60  0001 C CNN
 F 3 "" H 8100 3700 60  0000 C CNN
 	1    8100 3700
@@
 F 0 "K35" H 8850 3700 60  0000 C CNN
 F 1 "KEYSW" H 8900 3600 60  0001 C CNN
-F 2 "kudox_footprints:Mx_hotswappable" H 8900 3700 60  0001 C CNN
+F 2 "kudox_footprints:MX_reversible_100" H 8900 3700 60  0001 C CNN
 F 3 "" H 8900 3700 60  0000 C CNN
 	1    8900 3700
@@
 F 0 "K40" H 4850 4500 60  0000 C CNN
 F 1 "KEYSW" H 4900 4400 60  0001 C CNN
-F 2 "kudox_footprints:Mx_hotswappable" H 4900 4500 60  0001 C CNN
+F 2 "kudox_footprints:MX_reversible_100" H 4900 4500 60  0001 C CNN
 F 3 "" H 4900 4500 60  0000 C CNN
 	1    4900 4500
@@
 F 0 "K41" H 5650 4500 60  0000 C CNN
 F 1 "KEYSW" H 5700 4400 60  0001 C CNN
-F 2 "kudox_footprints:Mx_hotswappable" H 5700 4500 60  0001 C CNN
+F 2 "kudox_footprints:MX_reversible_100" H 5700 4500 60  0001 C CNN
 F 3 "" H 5700 4500 60  0000 C CNN
 	1    5700 4500
@@
 F 0 "K42" H 6450 4500 60  0000 C CNN
 F 1 "KEYSW" H 6500 4400 60  0001 C CNN
-F 2 "kudox_footprints:Mx_hotswappable" H 6500 4500 60  0001 C CNN
+F 2 "kudox_footprints:MX_reversible_100" H 6500 4500 60  0001 C CNN
 F 3 "" H 6500 4500 60  0000 C CNN
 	1    6500 4500
@@
 F 0 "K43" H 7250 4500 60  0000 C CNN
 F 1 "KEYSW" H 7300 4400 60  0001 C CNN
-F 2 "kudox_footprints:Mx_hotswappable" H 7300 4500 60  0001 C CNN
+F 2 "kudox_footprints:MX_reversible_100" H 7300 4500 60  0001 C CNN
 F 3 "" H 7300 4500 60  0000 C CNN
 	1    7300 4500
@@
 F 0 "K44" H 8050 4500 60  0000 C CNN
 F 1 "KEYSW" H 8100 4400 60  0001 C CNN
-F 2 "kudox_footprints:Mx_hotswappable" H 8100 4500 60  0001 C CNN
+F 2 "kudox_footprints:MX_reversible_100" H 8100 4500 60  0001 C CNN
 F 3 "" H 8100 4500 60  0000 C CNN
 	1    8100 4500
@@
 F 0 "K45" H 8850 4500 60  0000 C CNN
 F 1 "KEYSW" H 8900 4400 60  0001 C CNN
-F 2 "kudox_footprints:Mx_hotswappable" H 8900 4500 60  0001 C CNN
+F 2 "kudox_footprints:MX_reversible_100" H 8900 4500 60  0001 C CNN
 F 3 "" H 8900 4500 60  0000 C CNN
 	1    8900 4500
@@
 F 0 "K46" H 9650 4500 60  0000 C CNN
 F 1 "KEYSW" H 9700 4400 60  0001 C CNN
-F 2 "kudox_footprints:Mx_hotswappable" H 9700 4500 60  0001 C CNN
+F 2 "kudox_footprints:MX_reversible_100" H 9700 4500 60  0001 C CNN
 F 3 "" H 9700 4500 60  0000 C CNN
 	1    9700 4500
@@
 	8600 1900 9400 1900
 Connection ~ 8600 1900
+$Comp
+L Connector_Generic:Conn_01x01 J1
+U 1 1 60F83C68
+P 3000 3200
+F 0 "J1" H 3080 3242 50  0000 L CNN
+F 1 "RGB" H 3080 3151 50  0000 L CNN
+F 2 "kudox_footprints:pad_1x1" H 3000 3200 50  0001 C CNN
+F 3 "~" H 3000 3200 50  0001 C CNN
+	1    3000 3200
+	1    0    0    -1
+$EndComp
+Text GLabel 2650 3200 0    60   Input ~ 0
+SDA
+Wire Wire Line
+	2800 3200 2650 3200
+$Comp
+L Connector_Generic:Conn_01x01 J2
+U 1 1 60F96383
+P 3000 3450
+F 0 "J2" H 3080 3492 50  0000 L CNN
+F 1 "RGB" H 3080 3401 50  0000 L CNN
+F 2 "kudox_footprints:pad_1x1" H 3000 3450 50  0001 C CNN
+F 3 "~" H 3000 3450 50  0001 C CNN
+	1    3000 3450
+	1    0    0    -1
+$EndComp
+Text GLabel 2650 3450 0    60   Input ~ 0
+SDA
+Wire Wire Line
+	2800 3450 2650 3450
 $EndSCHEMATC
